File: Esp32PrinterController.kicad_pcb (KiCad board)
At the start: 2 copper layers, 157.5 x 97.8 mm, 101 parts, among them J1 -24V IN+, J10 +NOZ-, J11 +BED-, J110 MOT X, J12 +FAN1-, J13 +FAN2-, J14 +FAN3-, J20 +BT-, J21 +NT-, J23 MOT Y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

Commit message: Rev2, unbuilt
Parts:
- removed JP7: SolderJumper_2_Open, Jumper:SolderJumper-2_P1.3mm_Open_TrianglePad1.0x1.5mm
- added R1: 16.5k 1%, Resistor_THT:R_Axial_DIN0207_L6.3mm_D2.5mm_P10.16mm_Horizontal, F.Cu at (121.9, 101.0)
- added R2: 10k 1%, Resistor_THT:R_Axial_DIN0207_L6.3mm_D2.5mm_P10.16mm_Horizontal, F.Cu at (108.7, 102.9)
- added R3: 470, Resistor_THT:R_Axial_DIN0207_L6.3mm_D2.5mm_P10.16mm_Horizontal, F.Cu at (111.8, 97.8)
- added U7: TL431LP, Package_TO_SOT_THT:TO-92_Inline, F.Cu at (126.5, 100.8)
- added U8: 74LVC2G157, Package_SO:SSOP-8_2.95x2.8mm_P0.65mm, B.Cu at (145.5, 58.0)
- C3: moved to B.Cu
- J1, J10, J11, J12, J13, J14, J20, J21, J30, J31, J32: footprint this:PhoenixContact_MSTBVA_2,5_2-G-5,08_1x02_P5.08mm_Vertical_WallToWall -> Connector_Phoenix_MSTB:PhoenixContact_MSTBVA_2,5_2-G-5,08_1x02_P5.08mm_Vertical
- JP1: footprint Jumper:SolderJumper-3_P2.0mm_Open_TrianglePad1.0x1.5mm_NumberLabels -> Jumper:SolderJumper-3_P1.3mm_Open_RoundedPad1.0x1.5mm_NumberLabels
- Q1, Q2: footprint Package_TO_SOT_THT:TO-220-3_Vertical -> this:TO-220-3_Vertical_HeatSink
- moved JP23 26.2 mm to (145.0, 47.5), turned to 180 degrees
- moved JP24 17.4 mm to (145.0, 51.6), turned to 180 degrees
- moved F2 11.4 mm to (41.7, 117.3)
- moved D2 11.1 mm to (63.0, 79.5)
- moved D3 11.1 mm to (50.3, 79.5)
- moved R10 11.1 mm to (65.5, 93.5)
- moved R11 11.1 mm to (57.3, 87.1)
- moved R16 11.1 mm to (43.9, 86.5)
- moved R17 11.1 mm to (48.8, 83.3)
- moved R12 11.1 mm to (61.7, 83.3)
- moved R15 11.1 mm to (52.6, 93.5)
- moved Q1 6.86 mm to (63.0, 108.2), turned to 90 degrees
- moved Q2 5.59 mm to (51.6, 108.2), turned to 90 degrees
- moved C6 2.99 mm to (86.6, 42.2)
- moved C7 2.62 mm to (114.6, 42.2)
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Connections:
- net /Q139_E_EN renamed /Q141_E_EN
- net /Q141_E_DIR renamed /Q139_E_DIR
- A1 pad 13: /XYZ_MISO -> /STEP_MISO
- A2 pad 13: /XYZ_MISO -> /STEP_MISO
- A3 pad 13: /XYZ_MISO -> /STEP_MISO
- C3 pad 1: +3V3 -> /+3V3
- C4 pad 1: +3V3 -> /+3V3
- J60 pad 5: Net-(J60-Pad5) -> GND
- J60 pad 7: Net-(J60-Pad7) -> /IO16_BLSW
- JP1 pad 1: +3V3 -> /+3V3
- JP2 pad 1: /SD_MISO -> /STEP_MISO
- R20 pad 1: +3V3 -> /3.3Vreg
- R22 pad 1: +3V3 -> /3.3Vreg
- R30 pad 1: +3V3 -> /+3V3
- R31 pad 1: +3V3 -> /+3V3
- R32 pad 1: +3V3 -> /+3V3
- U1 pad 1: +3V3 -> /+3V3
- U1 pad 27: /SD_MISO -> /ESP_MISO
- U1 pad 31: Net-(U1-Pad31) -> /IO16_BLSW
- U6 pad 8: +3V3 -> /+3V3
Routing:
- net /SD_MISO: track 146.3 -> 23.2 mm, vias 0 -> 1
- net /STEP_MISO: track 0.00 -> 113.4 mm
- net /XYZ_MISO: track 109.6 -> 0.00 mm, vias 1 -> 0
- net /+3V3: track 0.00 -> 88.1 mm, vias 0 -> 1
- net +3V3: track 60.3 -> 0.00 mm
- net /IO16_BLSW: track 0.00 -> 52.5 mm, vias 0 -> 2
- net /Q142_FAN2: track 95.9 -> 44.6 mm, vias 0 -> 1
- net /XYZ_MS1: track 134.2 -> 88.6 mm, vias 0 -> 1
- net /Q143_FAN3: track 87.4 -> 42.1 mm, vias 0 -> 1
- net /PWR_IN: track 29.5 -> 0.00 mm
- net /XYZ_MS2: track 113.1 -> 87.1 mm
- net +24V2: track 23.2 -> 0.71 mm
- net /3.3Vreg: track 0.00 -> 21.8 mm
- net Net-(R1-Pad2): track 0.00 -> 20.7 mm
- net /SD_MOSI: track 186.8 -> 205.4 mm, vias 1 -> 3
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- added copper zone on F.Cu, net +24V2
- added copper zone on F.Cu, net /+3V3
- added copper zone on F.Cu, net /PWR_IN
- removed copper zone on F.Cu, net +3V3
Other:
- board text added: "+ 12-35V -"
- board text added: "E"
- board text added: "X"
- board text added: "Y"
- board text added: "Z"
