File: Esp32PrinterController.sch (KiCad schematic (older format))
At the start: 101 parts, among them J1 -24V IN+, J10 +NOZ-, J11 +BED-, J110 MOT X, J12 +FAN1-, J13 +FAN2-, J14 +FAN3-, J20 +BT-, J21 +NT-, J23 MOT Y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

Commit message: Added notes for next rev
Other:
- note added: "139_E_DIR"
- note added: "141_E_EN"
- note added: "C3 silkscreen outline too big"
- note added: "J1 silkscreen +- swapped"
- note added: "Level shifter for MISO"
- note added: "Make room for heatsinks on FETs"
- note added: "Move C110 to other side of Pololu"
- note added: "Move J110 farther from Pololu"
- note added: "R15 and R17 SWAPPED ON SILKSCREEN"
- note added: "Silkscreen labels for jumpers and stepper connectors"
- note added: "Voltage reference for thermistors TLVH431"
Changed lines of the file:
@@
 	1    0    0    -1
 $EndComp
+Text Notes 850  3550 0    100  ~ 20
+R15 and R17 SWAPPED ON SILKSCREEN
+Text Notes 12150 700  0    100  ~ 20
+Move J110 farther from Pololu
+Text Notes 13600 3350 0    100  ~ 20
+Move C110 to other side of Pololu
+Text Notes 2850 2750 0    100  ~ 20
+C3 silkscreen outline too big
+Text Notes 2100 4750 0    100  ~ 20
+Make room for heatsinks on FETs
+Text Notes 650  1400 0    100  ~ 20
+J1 silkscreen +- swapped
+Text Notes 10750 3900 0    70   ~ 14
+139_E_DIR
+Text Notes 10750 4100 0    70   ~ 14
+141_E_EN
+Text Notes 800  8350 0    100  ~ 20
+Silkscreen labels for jumpers and stepper connectors
+Text Notes 4650 3800 0    100  ~ 20
+Voltage reference for thermistors TLVH431
+Text Notes 10550 4850 0    100  ~ 20
+Level shifter for MISO
 $EndSCHEMATC

Commit message: Rev2, unbuilt
Parts:
- removed JP1: Jumper_3_Open, Jumper:SolderJumper-3_P2.0mm_Open_TrianglePad1.0x1.5mm_NumberLabels, symbol Jumper:Jumper_3_Open
- removed JP25: Jumper_3_Open, Jumper:SolderJumper-3_P1.3mm_Open_RoundedPad1.0x1.5mm_NumberLabels, symbol Jumper:Jumper_3_Open
- removed JP7: SolderJumper_2_Open, Jumper:SolderJumper-2_P1.3mm_Open_TrianglePad1.0x1.5mm, symbol Jumper:SolderJumper_2_Open
- added JP1, JP25: Jumper_3_Open, Jumper:SolderJumper-3_P1.3mm_Open_RoundedPad1.0x1.5mm_NumberLabels, symbol this:Jumper_3_Open
- added R1: 16.5k 1%, Resistor_THT:R_Axial_DIN0207_L6.3mm_D2.5mm_P10.16mm_Horizontal, symbol Device:R
- added R2: 10k 1%, Resistor_THT:R_Axial_DIN0207_L6.3mm_D2.5mm_P10.16mm_Horizontal, symbol Device:R
- added R3: 470, Resistor_THT:R_Axial_DIN0207_L6.3mm_D2.5mm_P10.16mm_Horizontal, symbol Device:R
- added U7: TL431LP, Package_TO_SOT_THT:TO-92_Inline, symbol Reference_Voltage:TL431LP
- added U8: 74LVC2G157, Package_SO:SSOP-8_2.95x2.8mm_P0.65mm, symbol this:74LVC2G157visVCC
Connections:
- net +3V3: now also JP1.1 (A), U8.8 (VCC); no longer R20.1, R22.1
- net +5V: now also JP1.3 (B), R3.1
- net CS_X: now also JP25.1 (A)
- net GND: now also J60.5 (Pin_5), R2.2, U7.2 (A), U8.4 (GND), U8.7 (~G)
- net SD_CS: now also U8.6 (~A~/B)
- net SD_MISO: now also U8.1 (A); no longer JP2.1 (A), U1.27 (IO19)
- net VCC: now also JP1.2 (C), JP25.3 (B)
- net at A1.12 (MS3): now also JP25.2 (C)
- net IO16_BLSW: now reaches J60.7 (Pin_7)
- net IO16_BLSW: now also U1.31 (IO16)
- net Q139_E_EN renamed Q141_E_EN
- net Q141_E_DIR renamed Q139_E_DIR
- net XYZ_MISO renamed STEP_MISO
- net STEP_MISO: now also JP2.1 (A), U8.2 (B)
- new net: R1.2, R2.1, U7.1 (REF)
- new net 3.3Vreg: R1.1, R20.1, R22.1, R3.2, U7.3 (K)
- new net ESP_MISO: U1.27 (IO19), U8.5 (Y)
- no-connect marks 31 -> 30
Other:
- note added: "D4 used as SCK for ST7920 serial mode"
- note added: "EN used as data (SDI)"
- note added: "RS used as CS"
- note removed: "139_E_DIR"
- note removed: "141_E_EN"
- note removed: "J1 silkscreen +- swapped"
- note removed: "Level shifter for MISO"
- note removed: "Make room for heatsinks on FETs"
- note removed: "Move C110 to other side of Pololu"
- note removed: "Move J110 farther from Pololu"
- note removed: "R15 and R17 SWAPPED ON SILKSCREEN"
- note removed: "Silkscreen labels for jumpers and stepper connectors"
- note removed: "Voltage reference for thermistors TLVH431"
